File: Hotglue Switch.kicad_sch (KiCad schematic)
At the start: 10 parts, among them J3 BATTERY, J8 +OUTPUT, J9 -OUTPUT, M1 Screw, M2 Screw

Commit message: commit of all modified files for rev 1.1, including gerbers, 3d step models, PCB, schematic, and project files.
Parts:
- D1: value 150060GS75003 -> XL-1608UBC-06A
- H1: value MountingHole -> M2 MountingHole; footprint MountingHole:MountingHole_3.2mm_M3_DIN965 -> MountingHole:MountingHole_2.2mm_M2_DIN965; now left out of the parts list
- H2: footprint Trent_Components_Library:screw_contact_3 -> Trent-footprints:Sinhoo-M1.6-screw-contact
- H4: value 9774010633R -> SMTSO1610MTJ; footprint Mounting_Wuerth:Mounting_Wuerth_WA-SMSI-M1.6_H1mm_9774010633 -> Trent-footprints:Mounting_Sinhoo_SMTSO1610MJT
- J3: footprint Trent_Components_Library:JST_XH_S3B-XH-A-1_1x03_P2.50mm_Horizontal_Aliexpress -> Trent-footprints:JST_XH_S3B-XH-A-1_1x03_P2.50mm_Horizontal_Aliexpress
- J8: footprint Trent_Components_Library:PinHeader_1x02_P2.54mm_Vertical Positive -> Trent-footprints:PinHeader_1x02_P2.54mm_Vertical Positive
- J9: footprint Trent_Components_Library:PinHeader_1x02_P2.54mm_Vertical Negative -> Trent-footprints:PinHeader_1x02_P2.54mm_Vertical Negative
- M1: value Screw -> M1.6 Screw; footprint Trent_Components_Library:Screw M1.6 -> Trent-footprints:Screw M1.6
- M2: value Screw -> M2 Screw; footprint Trent_Components_Library:Screw M3 -> Trent-footprints:Screw M2
- R1: value 560112140008 -> RC0603FR-07390RL; footprint Resistor_SMD:R_1210_3225Metric_Pad1.30x2.65mm_HandSolder -> Resistor_SMD:R_0603_1608Metric_Pad0.98x0.95mm_HandSolder
Changed lines of the file:
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@@
 (kicad_sch
-	(version 20231120)
+	(version 20250114)
 	(generator "eeschema")
-	(generator_version "8.0")
+	(generator_version "9.0")
 	(paper "A4")
 	(junction
@@
 		(at 38.1 48.26 0)
 		(unit 1)
-		(exclude_from_sim yes)
+		(exclude_from_sim no)
 		(in_bom no)
 		(on_board yes)
@@
 			)
 		)
-		(property "Value" "Screw"
+		(property "Value" "M2 Screw"
 			(at 40.64 49.5299 0)
 			(effects
@@
 			)
 		)
-		(property "Footprint" "Trent_Components_Library:Screw M3"
+		(property "Footprint" "Trent-footprints:Screw M2"
 			(at 38.1 48.26 0)
 			(effects
@@
 		(unit 1)
 		(exclude_from_sim no)
-		(in_bom yes)
+		(in_bom no)
 		(on_board yes)
 		(dnp no)
@@
 			)
 		)
-		(property "Value" "MountingHole"
+		(property "Value" "M2 MountingHole"
 			(at 40.64 39.37 0)
 			(effects
@@
 			)
 		)
-		(property "Footprint" "MountingHole:MountingHole_3.2mm_M3_DIN965"
+		(property "Footprint" "MountingHole:MountingHole_2.2mm_M2_DIN965"
 			(at 38.1 38.1 0)
 			(effects
@@
 			)
 		)
-		(property "Value" "150060GS75003"
+		(property "Value" "XL-1608UBC-06A"
 			(at 80.01 103.1875 90)
 			(effects
@@
 			)
 		)
-		(property "Datasheet" "~"
+		(property "Datasheet" "https://www.lcsc.com/datasheet/C7371904.pdf"
 			(at 76.2 100.33 0)
 			(effects
@@
 			)
 		)
-		(property "Description" "LED GREEN CLEAR 0603 SMD"
+		(property "Description" "LED BLUE WATER CLEAR 0603 SMD"
 			(at 76.2 100.33 0)
 			(effects
@@
 			)
 		)
-		(property "Footprint" "Trent_Components_Library:PinHeader_1x02_P2.54mm_Vertical Negative"
+		(property "Footprint" "Trent-footprints:PinHeader_1x02_P2.54mm_Vertical Negative"
 			(at 106.68 114.3 0)
 			(effects
@@
 			)
 		)
-		(property "Footprint" "Trent_Components_Library:JST_XH_S3B-XH-A-1_1x03_P2.50mm_Horizontal_Aliexpress"
+		(property "Footprint" "Trent-footprints:JST_XH_S3B-XH-A-1_1x03_P2.50mm_Horizontal_Aliexpress"
 			(at 38.1 68.58 0)
 			(effects
@@
 			)
 		)
-		(property "Footprint" "Trent_Components_Library:screw_contact_3"
+		(property "Footprint" "Trent-footprints:Sinhoo-M1.6-screw-contact"
 			(at 76.2 63.5 0)
 			(effects
@@
 			)
 		)
-		(property "Footprint" "Trent_Components_Library:PinHeader_1x02_P2.54mm_Vertical Positive"
+		(property "Footprint" "Trent-footprints:PinHeader_1x02_P2.54mm_Vertical Positive"
 			(at 106.68 78.74 0)
 			(effects
@@
 			)
 		)
-		(property "Value" "560112140008"
+		(property "Value" "RC0603FR-07390RL"
 			(at 78.74 90.17 0)
 			(effects
@@
 			)
 		)
-		(property "Footprint" "Resistor_SMD:R_1210_3225Metric_Pad1.30x2.65mm_HandSolder"
+		(property "Footprint" "Resistor_SMD:R_0603_1608Metric_Pad0.98x0.95mm_HandSolder"
 			(at 74.422 88.9 90)
 			(effects
@@
 			)
 		)
-		(property "Datasheet" "~"
+		(property "Datasheet" "https://www.lcsc.com/datasheet/C114620.pdf"
 			(at 76.2 88.9 0)
 			(effects
@@
 			)
 		)
-		(property "Description" "RES 220 OHM 5% 1/2W 1210"
+		(property "Description" "RES 390Ω ±1% 100mW 0603"
 			(at 76.2 88.9 0)
 			(effects
@@
 		(at 38.1 43.18 0)
 		(unit 1)
-		(exclude_from_sim yes)
+		(exclude_from_sim no)
 		(in_bom no)
 		(on_board yes)
@@
 			)
 		)
-		(property "Value" "Screw"
+		(property "Value" "M1.6 Screw"
 			(at 40.64 44.4499 0)
 			(effects
@@
 			)
 		)
-		(property "Footprint" "Trent_Components_Library:Screw M1.6"
+		(property "Footprint" "Trent-footprints:Screw M1.6"
 			(at 38.1 43.18 0)
 			(effects
@@
 		(at 76.2 73.66 0)
 		(unit 1)
-		(exclude_from_sim yes)
+		(exclude_from_sim no)
 		(in_bom no)
 		(on_board yes)
@@
 			)
 		)
-		(property "Value" "9774010633R"
+		(property "Value" "SMTSO1610MTJ"
 			(at 78.74 73.6599 0)
 			(effects
@@
 			)
 		)
-		(property "Footprint" "Mounting_Wuerth:Mounting_Wuerth_WA-SMSI-M1.6_H1mm_9774010633"
+		(property "Footprint" "Trent-footprints:Mounting_Sinhoo_SMTSO1610MJT"
 			(at 76.2 73.66 0)
 			(effects
@@
 		)
 	)
+	(embedded_fonts no)
 )
